File: Secondcansat.sch (KiCad schematic (older format))
At the start: 14 parts

Commit message: added everything
Parts:
- added C?: C, symbol Device:C
- added C? (x2): 100nF, symbol Device:C
- added C?: 1uF, symbol Device:C
- added C?: 4.7uF, symbol Device:C
- added IC?: XBP9B-XCWT-001, XBP9BXCWT001, symbol Cansat-rescue:XBP9B-XCWT-001
- added IMU?: BN0055breakout, symbol Cansat-rescue:IMUbreakout
- added J?: camerapower, symbol Connector_Generic:Conn_01x02
- added J?: OpenlogBreakout, symbol Connector_Generic:Conn_01x06
- added J?: Conn_02x03_Odd_Even, symbol Connector_Generic:Conn_02x03_Odd_Even
- added J?: CAM-M8Q-GPS, symbol Cansat-rescue:CAM-M8Q-GPS
- added J?: light sensor, symbol Connector_Generic:Conn_02x04_Counter_Clockwise
- added J?: MS5607, symbol Connector_Generic:Conn_02x04_Counter_Clockwise
- added Q?: Q_NMOS_DGS, symbol Device:Q_NMOS_DGS
- added R?: 10ohms, symbol Device:R
- added R? (x2): 2kohm, symbol Device:R
- added R? (x4): R, symbol Device:R
- added R?: 10kohm, symbol Device:R
- added REg?: 3.3vREG, symbol Connector_Generic:Conn_02x04_Counter_Clockwise
- added Servo?: Servo, symbol Connector_Generic:Conn_01x03
- added TH?: Thermistor, symbol Device:Thermistor
- added buzzer?: buzzer, symbol Connector_Generic:Conn_02x01
Connections:
- net labels added: ADCE0, CSB, IOPIN1, MISO, MOSI, PDICLK, PDIDATA, PWM, RX_OPenlog_PC2, RX_PD2, RX_PD6, SCL, SCLK, SDA, TX_PD3, TX_PD7, TX_openlog_PC3, Therm_ADCA0
- wire segments 36 -> 88
- no-connect marks 0 -> 6

Commit message: Finish schematic
Parts:
- added Moter?: Moter, symbol Connector_Generic:Conn_01x02
- added Q? (x4): Q_NMOS_DGS, symbol Device:Q_NMOS_DGS
- added R? (x8): 10kohm, symbol Device:R
Connections:
- net labels added: Moto2r_toggle1, Motor2_toggle2, Motor3_toggle3, Motor4_toggle4, Motor_toggle1, Motor_toggle2, Motor_toggle3, Motor_toggle4, TC_PD0
- net labels removed: IOPIN1
- wire segments 88 -> 145
- no-connect marks 6 -> 7

Commit message: fixed schematic and add breakout pcb comp
Connections:
- net labels removed: Motor3_toggle3, Motor4_toggle4, Motor_toggle3, Motor_toggle4
- wire segments 145 -> 146
Changed lines of the file:
@@
 $Descr A4 11693 8268
 encoding utf-8
-Sheet 1 14
+Sheet 1 15
 Title ""
 Date ""
@@
 Text GLabel 4150 1950 1    50   Input ~ 0
 Motor_toggle2
-Text GLabel 6400 1150 1    50   Input ~ 0
-Motor_toggle3
-Text GLabel 6500 1900 1    50   Input ~ 0
-Motor_toggle4
 $Comp
 L Device:R R?
@@
 Text GLabel 3350 4300 2    50   Input ~ 0
 Motor_toggle2
-Text GLabel 3350 4400 2    50   Input ~ 0
-Motor_toggle3
-Text GLabel 3350 4500 2    50   Input ~ 0
-Motor_toggle4
 Text GLabel 5850 7100 2    50   Input ~ 0
 TC_PD0
@@
 Text GLabel 8750 5850 1    50   Input ~ 0
 Motor2_toggle2
-Text GLabel 11000 5050 1    50   Input ~ 0
-Motor3_toggle3
-Text GLabel 11100 5800 1    50   Input ~ 0
-Motor4_toggle4
 $Comp
 L Device:R R?
@@
 Text GLabel 3350 4700 2    50   Input ~ 0
 Moto2r_toggle1
-Text GLabel 3350 4900 2    50   Input ~ 0
-Motor3_toggle3
-Text GLabel 3350 5000 2    50   Input ~ 0
-Motor4_toggle4
+$Comp
+L power:+3.3V #PWR?
+U 1 1 5C84969F
+P 11050 1300
+F 0 "#PWR?" H 11050 1150 50  0001 C CNN
+F 1 "+3.3V" V 11065 1428 50  0000 L CNN
+F 2 "" H 11050 1300 50  0001 C CNN
+F 3 "" H 11050 1300 50  0001 C CNN
+	1    11050 1300
+	0    1    1    0
+$EndComp
+Wire Wire Line
+	10900 1300 11050 1300
+Text GLabel 11000 5050 1    50   Input ~ 0
+Moto2r_toggle1
+Text GLabel 11100 5800 1    50   Input ~ 0
+Motor2_toggle2
+Text GLabel 6500 1900 1    50   Input ~ 0
+Motor_toggle2
+Text GLabel 6400 1150 1    50   Input ~ 0
+Motor_toggle1
 $EndSCHEMATC

Commit message: made pcb footprints
Parts:
- Battery1: renamed from Battery?; footprint (none) -> Connector_PinSocket_2.54mm:PinSocket_1x02_P2.54mm_Vertical
- C1, C2, C3, C4, C5, C6, C7, C8: renamed from C?; footprint (none) -> Capacitor_SMD:C_0603_1608Metric_Pad1.05x0.95mm_HandSolder
- IC1: renamed from IC?; footprint XBP9BXCWT001 -> CanSAT2ndtry:XBP9BXCWT001
- IMU1: renamed from IMU?; footprint (none) -> CanSAT2ndtry:BNO055breakout
- J1: renamed from J?; footprint (none) -> Connector_PinSocket_2.54mm:PinSocket_1x06_P2.54mm_Vertical
- J2: renamed from J?; footprint (none) -> Connector_PinSocket_2.54mm:PinSocket_1x02_P2.54mm_Vertical
- R12, R13, R14: renamed from R?; value R -> 10kohm
- buzzer1: renamed from buzzer?; footprint (none) -> Connector_PinSocket_2.54mm:PinSocket_1x03_P2.54mm_Vertical
- gave numbers to parts that had none: 36

Commit message: Added some part# and fixed H-bridges
Parts:
- removed Moter1: Moter, symbol Connector_Generic:Conn_01x02
- removed Q1, Q2, Q4, Q5, Q6, Q7, Q8, Q9: Q_NMOS_DGS, symbol Device:Q_NMOS_DGS
- removed R1, R10, R11, R15, R16, R2, R5, R6: 10kohm, symbol Device:R
- removed REg1: 3.3vREG, symbol Connector_Generic:Conn_02x04_Counter_Clockwise
- added C?: 1uF, symbol Device:C
- added C?: 50uF, symbol Device:C
- added Moter?: Moter_Adafruit_711, symbol Connector_Generic:Conn_01x02
- added R?: 2kohm, symbol Device:R
- added R? (x4): 10kohm, symbol Device:R
- added U? (x2): H-bridge_BD6210HFP-TR, symbol Cansat-rescue:H-bridge
- added VR?: VR__TLV75533PDBVR, symbol Cansat-rescue:VR__TLV75533PDBVR
- J4: value Conn_02x03_Odd_Even -> Debugger
- J5: value light sensor -> light_sensor__SFH 7776
- Moter?: renamed from Moter2; value Moter -> Moter_Adafruit_711
Connections:
- net labels added: ADC_A1, MoterRIN1, MoterRIN2, MotorFIN1, MotorFIN2
- net labels removed: Moto2r_toggle1, Motor2_toggle2, Motor_toggle1, Motor_toggle2
- wire segments 146 -> 128
- no-connect marks 7 -> 4

Commit message: Added footprints changed some schematic symbols
Parts:
- removed J3: MS5607, symbol Connector_Generic:Conn_02x04_Counter_Clockwise
- added J?: Pressure_MS5607, symbol Cansat-rescue:Pressure_MS5607
Changed lines of the file:
@@
 $Descr A4 11693 8268
 encoding utf-8
-Sheet 1 13
+Sheet 1 15
 Title ""
 Date ""
@@
 Text GLabel 3350 3800 2    50   Input ~ 0
 Therm_ADCA0
-$Comp
-L Connector_Generic:Conn_02x04_Counter_Clockwise J3
-U 1 1 5C8A3415
-P 7250 1950
-F 0 "J3" H 7300 2267 50  0000 C CNN
-F 1 "MS5607" H 7300 2176 50  0000 C CNN
-F 2 "" H 7250 1950 50  0001 C CNN
-F 3 "~" H 7250 1950 50  0001 C CNN
-	1    7250 1950
-	1    0    0    -1
-$EndComp
 $Comp
 L power:+3.3V #PWR037
@@
 Text GLabel 9300 5750 0    50   Input ~ 0
 MotorFIN2
+$Comp
+L Cansat-rescue:Pressure_MS5607 J?
+U 1 1 5C8FC930
+P 7250 1950
+F 0 "J?" H 7300 2275 50  0000 C CNN
+F 1 "Pressure_MS5607" H 7300 2184 50  0000 C CNN
+F 2 "" H 7250 1950 50  0001 C CNN
+F 3 "~" H 7250 1950 50  0001 C CNN
+	1    7250 1950
+	1    0    0    -1
+$EndComp
 $EndSCHEMATC

Commit message: Made sugested corrections
Parts:
- removed D1: DIODE, symbol pspice:DIODE
- removed MOSFET1: MOSFET N, symbol Device:Q_NMOS_DGS
- removed Moter?: Moter_Adafruit_711, symbol Connector_Generic:Conn_01x02
- removed R? (x2): 10kohm, symbol Device:R
- removed U? (x2): H-bridge_BD6210HFP-TR, symbol Cansat-rescue:H-bridge
- removed openlog1: openlog, symbol Connector_Generic:Conn_01x06
- added C2: 5uF, symbol Device:C
- added C5: 10uF, symbol Device:C
- added Moter1: Moter_Adafruit_711, symbol Connector_Generic:Conn_01x02
- added Q1: Q_PMOS_DGS, symbol Device:Q_PMOS_DGS
- added Q2: Q_NMOS_DGS, symbol Device:Q_NMOS_DGS
- added R1: 274kohm, symbol Device:R
- added R2: 30Kohm, symbol Device:R
- added R4, R5, R6: 10kohm, symbol Device:R
- added U1: VR_TPS7A7001DDAR, symbol Cansat-rescue:VR_TPS7A7001DDAR
- added U2, U3: H-bridge_MP6513GJ-P, symbol Cansat-rescue:H-bridge_MP6513GJ-P
- R11: renamed from R9; value R -> 10kohm
- R3: value 10ohms -> 10kohm
- R9: renamed from R7; value 2kohm -> 5kohm
- Servo1: value Servo -> Servo_Adafruit_1142
- gave numbers to parts that had none: 8
- renumbered C6 to C10, C7 to C11, C8 to C12, C2 to C3, C3 to C4, C4 to C7, C5 to C9, R12 to R14, R13 to R15, R14 to R16, R4 to R7
Connections:
- net labels added: +5V
- net labels removed: ADCE0
- wire segments 128 -> 124
- no-connect marks 4 -> 7

Commit message: Did the layout for PCB now Just need to do traces
Parts:
- added C1: CP1, Capacitor_SMD:C_1206_3216Metric_Pad1.42x1.75mm_HandSolder, symbol Device:CP1
- added L2: INDUCTOR, Inductor_SMD:L_0805_2012Metric_Pad1.15x1.40mm_HandSolder, symbol pspice:INDUCTOR
- C3: renamed from C2; footprint (none) -> Capacitor_SMD:C_0603_1608Metric_Pad1.05x0.95mm_HandSolder
- C4: renamed from C3; value C -> 100nF
- C5: renamed from C4; footprint Capacitor_SMD:C_0603_1608Metric_Pad1.05x0.95mm_HandSolder -> Capacitor_SMD:C_1206_3216Metric_Pad1.42x1.75mm_HandSolder
- C6: renamed from C5; footprint (none) -> Capacitor_SMD:C_0805_2012Metric_Pad1.15x1.40mm_HandSolder
- C7: renamed from C6; footprint (none) -> Capacitor_SMD:C_0603_1608Metric_Pad1.05x0.95mm_HandSolder
- C8: renamed from C7; value C -> 1uF
- C9: renamed from C8; footprint (none) -> Capacitor_SMD:C_1206_3216Metric_Pad1.42x1.75mm_HandSolder
- J3: footprint (none) -> CanSAT2ndtry:MS5607
- J4: footprint (none) -> Connector_PinSocket_2.54mm:PinSocket_2x03_P2.54mm_Vertical
- J5: footprint (none) -> Connector_PinSocket_2.54mm:PinSocket_2x04_P2.54mm_Vertical
- J6: footprint (none) -> CanSAT2ndtry:CAM-M8Q
- L1: footprint (none) -> Inductor_SMD:L_0805_2012Metric_Pad1.15x1.40mm_HandSolder
- MCU1: footprint Package_QFP:TQFP-44_10x10mm_P0.8mm -> CanSAT2ndtry:ATXMEGA128A4U-AU
- Moter1, Moter2: footprint (none) -> Connector_PinHeader_2.54mm:PinHeader_2x01_P2.54mm_Vertical
- Q1, Q2, Q3: footprint (none) -> Package_TO_SOT_SMD:SOT-23
- R1: footprint (none) -> Resistor_SMD:R_1206_3216Metric
- R10, R8, R9: footprint (none) -> Capacitor_SMD:C_0805_2012Metric
- R11, R12, R13, R14, R15, R16, R3, R4, R5, R6, R7: footprint (none) -> Resistor_SMD:R_0603_1608Metric_Pad1.05x0.95mm_HandSolder
- R2: footprint (none) -> Resistor_SMD:R_0805_2012Metric_Pad1.15x1.40mm_HandSolder
- Servo1: footprint (none) -> Connector_PinSocket_2.54mm:PinSocket_1x03_P2.54mm_Vertical
- TH1: footprint (none) -> Connector_PinSocket_2.54mm:PinSocket_2x01_P2.54mm_Vertical
- U1: footprint (none) -> CanSAT2ndtry:VR_TPS7A7001DDAR
- U2, U3: footprint (none) -> CanSAT2ndtry:H-Bridge_MP6513GJ-P
- VR1: footprint (none) -> CanSAT2ndtry:VR_296-50411-1-ND
- renumbered C9 to C10, C10 to C11, C11 to C12, C12 to C13, C1 to C2
Connections:
- wire segments 124 -> 126
