File: Secondcansat.sch (KiCad schematic (older format))
At the start: 53 parts, among them IC1 XBP9B-XCWT-001, J1 OpenlogBreakout, J2 camerapower, J3 Pressure_MS5607, J4 Debugger, J5 light_sensor__SFH 7776, J6 CAM-M8Q-GPS, Q1 Q_PMOS_DGS, Q2 Q_NMOS_DGS, Q3 Q_NMOS_DGS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

Commit message: added prototype pins
Parts:
- added J10: SDA, Connector_PinSocket_2.54mm:PinSocket_1x01_P2.54mm_Vertical, symbol Connector_Generic:Conn_01x01
- added J11: 5V, Connector_PinSocket_2.54mm:PinSocket_1x01_P2.54mm_Vertical, symbol Connector_Generic:Conn_01x01
- added J12: Tx, Connector_PinSocket_2.54mm:PinSocket_1x01_P2.54mm_Vertical, symbol Connector_Generic:Conn_01x01
- added J13: Rx, Connector_PinSocket_2.54mm:PinSocket_1x01_P2.54mm_Vertical, symbol Connector_Generic:Conn_01x01
- added J7: GND, Connector_PinSocket_2.54mm:PinSocket_1x01_P2.54mm_Vertical, symbol Connector_Generic:Conn_01x01
- added J8: SCL, Connector_PinSocket_2.54mm:PinSocket_1x01_P2.54mm_Vertical, symbol Connector_Generic:Conn_01x01
- added J9: 3v, Connector_PinSocket_2.54mm:PinSocket_1x01_P2.54mm_Vertical, symbol Connector_Generic:Conn_01x01
- buzzer1: footprint Connector_PinSocket_2.54mm:PinSocket_1x03_P2.54mm_Vertical -> Connector_PinSocket_2.54mm:PinSocket_1x02_P2.54mm_Vertical
Changed lines of the file:
@@
 F 0 "buzzer1" H 6300 7467 50  0000 C CNN
 F 1 "buzzer" H 6300 7400 50  0000 C CNN
-F 2 "Connector_PinSocket_2.54mm:PinSocket_1x03_P2.54mm_Vertical" H 6250 7250 50  0001 C CNN
+F 2 "Connector_PinSocket_2.54mm:PinSocket_1x02_P2.54mm_Vertical" H 6250 7250 50  0001 C CNN
 F 3 "~" H 6250 7250 50  0001 C CNN
 	1    6250 7250
@@
 	1550 7200 1250 7200
 Connection ~ 1250 7200
+$Comp
+L Connector_Generic:Conn_01x01 J9
+U 1 1 5C92ECB5
+P 7750 5850
+F 0 "J9" V 7623 5930 50  0000 L CNN
+F 1 "3v" V 7714 5930 50  0000 L CNN
+F 2 "Connector_PinSocket_2.54mm:PinSocket_1x01_P2.54mm_Vertical" H 7750 5850 50  0001 C CNN
+F 3 "~" H 7750 5850 50  0001 C CNN
+	1    7750 5850
+	0    1    1    0
+$EndComp
+$Comp
+L Connector_Generic:Conn_01x01 J10
+U 1 1 5C92EE16
+P 7950 6250
+F 0 "J10" V 7823 6330 50  0000 L CNN
+F 1 "SDA" V 7914 6330 50  0000 L CNN
+F 2 "Connector_PinSocket_2.54mm:PinSocket_1x01_P2.54mm_Vertical" H 7950 6250 50  0001 C CNN
+F 3 "~" H 7950 6250 50  0001 C CNN
+	1    7950 6250
+	0    1    1    0
+$EndComp
+$Comp
+L Connector_Generic:Conn_01x01 J8
+U 1 1 5C92EE9C
+P 7550 6300
+F 0 "J8" V 7423 6380 50  0000 L CNN
+F 1 "SCL" V 7514 6380 50  0000 L CNN
+F 2 "Connector_PinSocket_2.54mm:PinSocket_1x01_P2.54mm_Vertical" H 7550 6300 50  0001 C CNN
+F 3 "~" H 7550 6300 50  0001 C CNN
+	1    7550 6300
+	0    1    1    0
+$EndComp
+$Comp
+L Connector_Generic:Conn_01x01 J7
+U 1 1 5C92EF26
+P 7300 5850
+F 0 "J7" V 7173 5930 50  0000 L CNN
+F 1 "GND" V 7264 5930 50  0000 L CNN
+F 2 "Connector_PinSocket_2.54mm:PinSocket_1x01_P2.54mm_Vertical" H 7300 5850 50  0001 C CNN
+F 3 "~" H 7300 5850 50  0001 C CNN
+	1    7300 5850
+	0    1    1    0
+$EndComp
+$Comp
+L Connector_Generic:Conn_01x01 J11
+U 1 1 5C930677
+P 8150 5900
+F 0 "J11" V 8023 5980 50  0000 L CNN
+F 1 "5V" V 8114 5980 50  0000 L CNN
+F 2 "Connector_PinSocket_2.54mm:PinSocket_1x01_P2.54mm_Vertical" H 8150 5900 50  0001 C CNN
+F 3 "~" H 8150 5900 50  0001 C CNN
+	1    8150 5900
+	0    1    1    0
+$EndComp
+$Comp
+L Connector_Generic:Conn_01x01 J12
+U 1 1 5C9313B4
+P 8450 6250
+F 0 "J12" V 8323 6330 50  0000 L CNN
+F 1 "Tx" V 8414 6330 50  0000 L CNN
+F 2 "Connector_PinSocket_2.54mm:PinSocket_1x01_P2.54mm_Vertical" H 8450 6250 50  0001 C CNN
+F 3 "~" H 8450 6250 50  0001 C CNN
+	1    8450 6250
+	0    1    1    0
+$EndComp
+$Comp
+L Connector_Generic:Conn_01x01 J13
+U 1 1 5C931444
+P 8700 6000
+F 0 "J13" V 8573 6080 50  0000 L CNN
+F 1 "Rx" V 8664 6080 50  0000 L CNN
+F 2 "Connector_PinSocket_2.54mm:PinSocket_1x01_P2.54mm_Vertical" H 8700 6000 50  0001 C CNN
+F 3 "~" H 8700 6000 50  0001 C CNN
+	1    8700 6000
+	0    1    1    0
+$EndComp
+Text GLabel 7950 6050 1    50   Input ~ 0
+SDA
+Text GLabel 7550 6100 1    50   Input ~ 0
+SCL
+Text GLabel 8700 5800 1    50   Input ~ 0
+RX_PD6
+Text GLabel 8450 6050 1    50   Input ~ 0
+TX_PD7
+$Comp
+L power:GND #PWR0101
+U 1 1 5C9348F6
+P 7300 5650
+F 0 "#PWR0101" H 7300 5400 50  0001 C CNN
+F 1 "GND" H 7305 5477 50  0000 C CNN
+F 2 "" H 7300 5650 50  0001 C CNN
+F 3 "" H 7300 5650 50  0001 C CNN
+	1    7300 5650
+	-1   0    0    1
+$EndComp
+$Comp
+L power:+3.3V #PWR0102
+U 1 1 5C9349F1
+P 7750 5650
+F 0 "#PWR0102" H 7750 5500 50  0001 C CNN
+F 1 "+3.3V" H 7765 5823 50  0000 C CNN
+F 2 "" H 7750 5650 50  0001 C CNN
+F 3 "" H 7750 5650 50  0001 C CNN
+	1    7750 5650
+	1    0    0    -1
+$EndComp
+$Comp
+L power:+5V #PWR0103
+U 1 1 5C934A7D
+P 8150 5700
+F 0 "#PWR0103" H 8150 5550 50  0001 C CNN
+F 1 "+5V" H 8165 5873 50  0000 C CNN
+F 2 "" H 8150 5700 50  0001 C CNN
+F 3 "" H 8150 5700 50  0001 C CNN
+	1    8150 5700
+	1    0    0    -1
+$EndComp
 $EndSCHEMATC

Commit message: Made some fixes to the PCB and footprint
Parts:
- removed Battery1: battery, Connector_PinSocket_2.54mm:PinSocket_1x02_P2.54mm_Vertical, symbol Connector_Generic:Conn_01x02
- removed J5: light_sensor__SFH 7776, Connector_PinSocket_2.54mm:PinSocket_2x04_P2.54mm_Vertical, symbol Connector_Generic:Conn_02x04_Counter_Clockwise
- added C14: 5uF, Capacitor_SMD:C_0603_1608Metric_Pad1.05x0.95mm_HandSolder, symbol Device:C
- added J14: Battery_Holder_keystone 1079, CanSAT2ndtry:BatteryHolder, symbol Cansat-rescue:Battery_Holder
- added J5: SFH_7776_OSRAM, CanSAT2ndtry:SFH7776, symbol Cansat-rescue:SFH_7776_OSRAM
- added Q4: Q_NMOS_BSS138, Package_TO_SOT_SMD:SOT-23, symbol Device:Q_NMOS_DGS
- added R17: 10kohm, Resistor_SMD:R_0603_1608Metric_Pad1.05x0.95mm_HandSolder, symbol Device:R
- added R18, R19: 220ohm, Resistor_SMD:R_0603_1608Metric_Pad1.05x0.95mm_HandSolder, symbol Device:R
- C1, C5: value CP1 -> 10uF
- C2: value C -> 100nF
- IC1: footprint CanSAT2ndtry:XBP9BXCWT001 -> CanSAT2ndtry:XBP9BXCWT001_2
- J4: footprint Connector_PinSocket_2.54mm:PinSocket_2x03_P2.54mm_Vertical -> Connector_PinSocket_1.27mm:PinSocket_2x03_P1.27mm_Vertical
- L1, L2: value INDUCTOR -> 10uH
- Q1: value Q_PMOS_DGS -> Q_PMOS_DMG2305UX-13DIDKR-ND
- Q2, Q3: value Q_NMOS_DGS -> Q_NMOS_BSS138
- TH1: value Thermistor -> Therm_NXRT15WB473FA3A016
- buzzer1: value buzzer -> buzzer_MAS803Q
Connections:
- net labels added: INT, cameraon
- net labels removed: RX_OPenlog_PC2, TX_openlog_PC3
- wire segments 126 -> 141

Commit message: added pull down resistors
Parts:
- removed J2: camerapower, Connector_PinSocket_2.54mm:PinSocket_1x02_P2.54mm_Vertical, symbol Connector_Generic:Conn_01x02
- added J2: Camera, Connector_PinSocket_2.54mm:PinSocket_1x03_P2.54mm_Vertical, symbol Connector_Generic:Conn_01x03
- added R20: 10kohm, Resistor_SMD:R_0603_1608Metric_Pad1.05x0.95mm_HandSolder, symbol Device:R
Changed lines of the file:
@@
 USART_RX_PC2
-$Comp
-L Connector_Generic:Conn_01x02 J2
-U 1 1 5C83BAE9
-P 5700 2700
-F 0 "J2" V 5573 2780 50  0000 L CNN
-F 1 "camerapower" V 5664 2780 50  0000 L CNN
-F 2 "Connector_PinSocket_2.54mm:PinSocket_1x02_P2.54mm_Vertical" H 5700 2700 50  0001 C CNN
-F 3 "~" H 5700 2700 50  0001 C CNN
-	1    5700 2700
-	0    -1   -1   0
-$EndComp
 $Comp
 L power:GND #PWR032
@@
 P 5800 2900
 F 0 "#PWR033" H 5800 2750 50  0001 C CNN
-F 1 "+5V" H 5815 3073 50  0000 C CNN
+F 1 "+5V" H 5750 3100 50  0000 C CNN
 F 2 "" H 5800 2900 50  0001 C CNN
 F 3 "" H 5800 2900 50  0001 C CNN
@@
 Wire Wire Line
 	1050 900  1050 1250
+$Comp
+L Connector_Generic:Conn_01x03 J2
+U 1 1 5C99FF9D
+P 5800 2700
+F 0 "J2" V 5766 2512 50  0000 R CNN
+F 1 "Camera" V 5675 2512 50  0000 R CNN
+F 2 "Connector_PinSocket_2.54mm:PinSocket_1x03_P2.54mm_Vertical" H 5800 2700 50  0001 C CNN
+F 3 "~" H 5800 2700 50  0001 C CNN
+	1    5800 2700
+	0    -1   -1   0
+$EndComp
+$Comp
+L power:GND #PWR0105
+U 1 1 5C9A036D
+P 5900 2900
+F 0 "#PWR0105" H 5900 2650 50  0001 C CNN
+F 1 "GND" H 6050 2800 50  0000 C CNN
+F 2 "" H 5900 2900 50  0001 C CNN
+F 3 "" H 5900 2900 50  0001 C CNN
+	1    5900 2900
+	1    0    0    -1
+$EndComp
+$Comp
+L Device:R R20
+U 1 1 5C9AF8E3
+P 5400 2950
+F 0 "R20" H 5470 2996 50  0000 L CNN
+F 1 "10kohm" H 5470 2905 50  0000 L CNN
+F 2 "Resistor_SMD:R_0603_1608Metric_Pad1.05x0.95mm_HandSolder" V 5330 2950 50  0001 C CNN
+F 3 "~" H 5400 2950 50  0001 C CNN
+	1    5400 2950
+	1    0    0    -1
+$EndComp
+$Comp
+L power:GND #PWR0106
+U 1 1 5C9B5798
+P 5400 2800
+F 0 "#PWR0106" H 5400 2550 50  0001 C CNN
+F 1 "GND" H 5405 2627 50  0000 C CNN
+F 2 "" H 5400 2800 50  0001 C CNN
+F 3 "" H 5400 2800 50  0001 C CNN
+	1    5400 2800
+	-1   0    0    1
+$EndComp
 $EndSCHEMATC

Commit message: changed footprint for Osram
Parts:
- J5: footprint CanSAT2ndtry:SFH7776 -> Connector_PinSocket_2.00mm:PinSocket_2x04_P2.00mm_Vertical
Changed lines of the file:
@@
 F 0 "J5" H 10000 3350 50  0000 C CNN
 F 1 "SFH_7776_OSRAM" H 9950 4550 50  0000 C CNN
-F 2 "CanSAT2ndtry:SFH7776" H 10100 3550 50  0001 C CNN
+F 2 "Connector_PinSocket_2.00mm:PinSocket_2x04_P2.00mm_Vertical" H 10100 3550 50  0001 C CNN
 F 3 "~" H 10100 3550 50  0001 C CNN
 	1    10050 3650

Commit message: added backup power and usb mini connector
Parts:
- added J15: USB_B_Mini, CanSAT2ndtry:USB-Mini, symbol Connector:USB_B_Mini
- added J16: coinBattery, CanSAT2ndtry:coin_Battery_120591-1, symbol Cansat-rescue:coinBattery
Connections:
- wire segments 141 -> 153
Changed lines of the file:
@@
 $Descr A4 11693 8268
 encoding utf-8
-Sheet 1 9
+Sheet 1 8
 Title ""
 Date ""
@@
 $EndComp
 $Comp
-L power:+6V #PWR014
-U 1 1 5C86EFA0
-P 4500 6950
-F 0 "#PWR014" H 4500 6800 50  0001 C CNN
-F 1 "+6V" V 4515 7078 50  0000 L CNN
-F 2 "" H 4500 6950 50  0001 C CNN
-F 3 "" H 4500 6950 50  0001 C CNN
-	1    4500 6950
-	0    -1   -1   0
-$EndComp
-$Comp
 L Connector_Generic:Conn_02x01 buzzer1
 U 1 1 5C872BCE
-P 6250 7250
-F 0 "buzzer1" H 6300 7467 50  0000 C CNN
-F 1 "buzzer_MAS803Q" H 6300 7400 50  0000 C CNN
-F 2 "Connector_PinSocket_2.54mm:PinSocket_1x02_P2.54mm_Vertical" H 6250 7250 50  0001 C CNN
-F 3 "~" H 6250 7250 50  0001 C CNN
-	1    6250 7250
+P 6550 7000
+F 0 "buzzer1" H 6600 7217 50  0000 C CNN
+F 1 "buzzer_MAS803Q" H 6600 7150 50  0000 C CNN
+F 2 "Connector_PinSocket_2.54mm:PinSocket_1x02_P2.54mm_Vertical" H 6550 7000 50  0001 C CNN
+F 3 "~" H 6550 7000 50  0001 C CNN
+	1    6550 7000
 	1    0    0    -1
 $EndComp
@@
 L Device:Q_NMOS_DGS Q3
 U 1 1 5C873B36
-P 5850 7150
-F 0 "Q3" V 6193 7150 50  0000 C CNN
-F 1 "Q_NMOS_BSS138" V 6102 7150 50  0000 C CNN
-F 2 "Package_TO_SOT_SMD:SOT-23" H 6050 7250 50  0001 C CNN
-F 3 "~" H 5850 7150 50  0001 C CNN
-	1    5850 7150
+P 6150 6900
+F 0 "Q3" V 6493 6900 50  0000 C CNN
+F 1 "Q_NMOS_BSS138" V 6402 6900 50  0000 C CNN
+F 2 "Package_TO_SOT_SMD:SOT-23" H 6350 7000 50  0001 C CNN
+F 3 "~" H 6150 6900 50  0001 C CNN
+	1    6150 6900
 	0    1    1    0
 $EndComp
@@
 L Device:R R7
 U 1 1 5C875FDE
-P 5850 6700
-F 0 "R7" H 5780 6654 50  0000 R CNN
-F 1 "10kohm" H 5780 6745 50  0000 R CNN
-F 2 "Resistor_SMD:R_0603_1608Metric_Pad1.05x0.95mm_HandSolder" V 5780 6700 50  0001 C CNN
-F 3 "~" H 5850 6700 50  0001 C CNN
-	1    5850 6700
+P 6150 6450
+F 0 "R7" H 6080 6404 50  0000 R CNN
+F 1 "10kohm" H 6080 6495 50  0000 R CNN
+F 2 "Resistor_SMD:R_0603_1608Metric_Pad1.05x0.95mm_HandSolder" V 6080 6450 50  0001 C CNN
+F 3 "~" H 6150 6450 50  0001 C CNN
+	1    6150 6450
 	1    0    0    -1
 $EndComp
@@
 L power:+6V #PWR035
 U 1 1 5C87605F
-P 6550 7250
-F 0 "#PWR035" H 6550 7100 50  0001 C CNN
-F 1 "+6V" V 6565 7378 50  0000 L CNN
-F 2 "" H 6550 7250 50  0001 C CNN
-F 3 "" H 6550 7250 50  0001 C CNN
-	1    6550 7250
+P 6850 7000
+F 0 "#PWR035" H 6850 6850 50  0001 C CNN
+F 1 "+6V" V 6865 7128 50  0000 L CNN
+F 2 "" H 6850 7000 50  0001 C CNN
+F 3 "" H 6850 7000 50  0001 C CNN
+	1    6850 7000
 	0    1    1    0
 $EndComp
@@
 L power:GND #PWR031
 U 1 1 5C8760E2
-P 5650 7250
-F 0 "#PWR031" H 5650 7000 50  0001 C CNN
-F 1 "GND" V 5655 7122 50  0000 R CNN
-F 2 "" H 5650 7250 50  0001 C CNN
-F 3 "" H 5650 7250 50  0001 C CNN
-	1    5650 7250
+P 5950 7000
+F 0 "#PWR031" H 5950 6750 50  0001 C CNN
+F 1 "GND" V 5955 6872 50  0000 R CNN
+F 2 "" H 5950 7000 50  0001 C CNN
+F 3 "" H 5950 7000 50  0001 C CNN
+	1    5950 7000
 	0    1    1    0
 $EndComp
@@
 L power:GND #PWR034
 U 1 1 5C876351
-P 5850 6550
-F 0 "#PWR034" H 5850 6300 50  0001 C CNN
-F 1 "GND" H 5700 6500 50  0000 C CNN
-F 2 "" H 5850 6550 50  0001 C CNN
-F 3 "" H 5850 6550 50  0001 C CNN
-	1    5850 6550
+P 6150 6300
+F 0 "#PWR034" H 6150 6050 50  0001 C CNN
+F 1 "GND" H 6000 6250 50  0000 C CNN
+F 2 "" H 6150 6300 50  0001 C CNN
+F 3 "" H 6150 6300 50  0001 C CNN
+	1    6150 6300
 	-1   0    0    1
 $EndComp
@@
 Text GLabel 3350 4300 2    50   Input ~ 0
 MoterRIN2
-Text GLabel 5850 6900 0    50   Input ~ 0
+Text GLabel 6150 6650 0    50   Input ~ 0
 TC_PD0
 Text GLabel 1950 5200 0    50   Input ~ 0
@@
 NoConn ~ 7550 2150
 Wire Wire Line
-	5850 6950 5850 6850
+	6150 6700 6150 6600
 $Comp
 L Connector_Generic:Conn_01x02 Moter2
@@
 F 3 "~" H 4550 6800 50  0001 C CNN
 	1    4550 6800
-	1    0    0    -1
-$EndComp
-Wire Wire Line
-	4500 6950 4550 6950
+	1    0    0    1
+$EndComp
 Connection ~ 4550 6950
 Wire Wire Line
@@
 	0    1    1    0
 $EndComp
-$Sheet
-S 4250 6450 1100 1050
-U 5C8EC4ED
-F0 "Sheet5C8EC4EC" 50
-F1 "VoltageRegsch.sch" 50
-$EndSheet
 $Comp
 L power:GND #PWR051
@@
 	-1   0    0    1
 $EndComp
+$Comp
+L Cansat-rescue:coinBattery J16
+U 1 1 5C9F0A92
+P 8500 1550
+F 0 "J16" H 8420 1875 50  0000 C CNN
+F 1 "coinBattery" H 8420 1784 50  0000 C CNN
+F 2 "CanSAT2ndtry:coin_Battery_120591-1" H 8500 1550 50  0001 C CNN
+F 3 "~" H 8500 1550 50  0001 C CNN
+	1    8500 1550
+	-1   0    0    -1
+$EndComp
+$Comp
+L Connector:USB_B_Mini J15
+U 1 1 5C9F0C34
+P 5600 7600
+F 0 "J15" V 5702 7930 50  0000 L CNN
+F 1 "USB_B_Mini" V 5611 7930 50  0000 L CNN
+F 2 "CanSAT2ndtry:USB-Mini" H 5750 7550 50  0001 C CNN
+F 3 "~" H 5750 7550 50  0001 C CNN
+	1    5600 7600
+	0    -1   -1   0
+$EndComp
+$Comp
+L power:+5V #PWR0107
+U 1 1 5C9FC88C
+P 4400 6950
+F 0 "#PWR0107" H 4400 6800 50  0001 C CNN
+F 1 "+5V" H 4415 7123 50  0000 C CNN
+F 2 "" H 4400 6950 50  0001 C CNN
+F 3 "" H 4400 6950 50  0001 C CNN
+	1    4400 6950
+	0    -1   -1   0
+$EndComp
+Wire Wire Line
+	5400 7300 5200 7300
+Wire Wire Line
+	5200 7300 5200 7400
+Wire Wire Line
+	5200 7400 4450 7400
+Wire Wire Line
+	4450 7400 4450 6950
+Wire Wire Line
+	4450 6950 4550 6950
+Wire Wire Line
+	4400 6950 4450 6950
+Connection ~ 4450 6950
+$Comp
+L power:GND #PWR0108
+U 1 1 5CA14814
+P 6000 7600
+F 0 "#PWR0108" H 6000 7350 50  0001 C CNN
+F 1 "GND" V 6005 7472 50  0000 R CNN
+F 2 "" H 6000 7600 50  0001 C CNN
+F 3 "" H 6000 7600 50  0001 C CNN
+	1    6000 7600
+	0    -1   -1   0
+$EndComp
+Wire Wire Line
+	8700 1550 8700 1600
+Wire Wire Line
+	8700 1600 8850 1600
+Wire Wire Line
+	8850 1600 8850 550
+Wire Wire Line
+	8850 550  11200 550
+Wire Wire Line
+	11200 550  11200 1400
+Wire Wire Line
+	11200 1400 10900 1400
+Connection ~ 8700 1600
+Wire Wire Line
+	8700 1600 8700 1650
+$Comp
+L power:GND #PWR?
+U 1 1 5CA36EA2
+P 8700 1450
+F 0 "#PWR?" H 8700 1200 50  0001 C CNN
+F 1 "GND" V 8705 1322 50  0000 R CNN
+F 2 "" H 8700 1450 50  0001 C CNN
+F 3 "" H 8700 1450 50  0001 C CNN
+	1    8700 1450
+	0    -1   -1   0
+$EndComp
 $EndSCHEMATC
